File: HW2/ME433HW2/433hw2.brd (EAGLE design)
At the start: 50 x 50 mm, 19 parts

Commit message: layout
Parts:
- moved LED2 59.4 mm to (43.2, 2.54), turned to 0 degrees
- moved R4 51.1 mm to (47.0, 6.35), turned to 270 degrees
- moved J1 21.6 mm to (21.6, 44.5), turned to 0 degrees
- moved C1 7.62 mm to (38.1, 3.81)
- moved U$5 5.39 mm to (41.9, 8.89)
- moved R1 5.08 mm to (15.2, 44.5)
- moved C3 3.81 mm to (15.2, 47.0), turned to 180 degrees
Routing:
- net N$10: track 29.7 -> 41.2 mm
- net N$26: track 10.5 -> 21.1 mm
- net N$11: track 31.5 -> 23.9 mm
- net N$8: track 0.00 -> 5.08 mm
- net N$9: track 0.00 -> 2.54 mm
Changed lines of the file:
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@@
 </autorouter>
 <elements>
-<element name="C1" library="433LIB" package="E2,5-6" value="" x="45.72" y="3.81" rot="R90"/>
-<element name="C3" library="433LIB" package="C025-025X050" value="" x="15.24" y="43.18"/>
+<element name="C1" library="433LIB" package="E2,5-6" value="" x="38.1" y="3.81" rot="R90"/>
+<element name="C3" library="433LIB" package="C025-025X050" value="" x="15.24" y="46.99" rot="R180"/>
 <element name="C4" library="433LIB" package="C025-025X050" value="" x="11.43" y="19.05" rot="R270"/>
 <element name="IC1" library="433LIB" package="DIL28-4" value="" x="27.94" y="21.59" rot="R270"/>
-<element name="J1" library="433LIB" package="1X05" value="" x="11.43" y="25.4" rot="R90"/>
+<element name="J1" library="433LIB" package="1X05" value="" x="21.59" y="44.45"/>
 <element name="J2" library="433LIB" package="1X08_ROUND" value="" x="16.51" y="17.78" rot="R90">
 <attribute name="PROD_ID" value="CONN-08437" x="16.51" y="17.78" size="1.778" layer="27" rot="R90" display="off"/>
@@
 </element>
 <element name="LED1" library="433LIB" package="LED3MM" value="" x="3.81" y="6.35" rot="R270"/>
-<element name="LED2" library="433LIB" package="LED3MM" value="" x="3.81" y="46.99" rot="R90"/>
-<element name="R1" library="433LIB" package="0207/7" value="" x="15.24" y="39.37"/>
+<element name="LED2" library="433LIB" package="LED3MM" value="" x="43.18" y="2.54"/>
+<element name="R1" library="433LIB" package="0207/7" value="" x="15.24" y="44.45"/>
 <element name="R2" library="433LIB" package="0207/7" value="" x="15.24" y="5.08" rot="R180"/>
 <element name="R3" library="433LIB" package="0207/7" value="" x="15.24" y="2.54"/>
-<element name="R4" library="433LIB" package="0207/7" value="" x="17.78" y="48.26" rot="R180"/>
+<element name="R4" library="433LIB" package="0207/7" value="" x="46.99" y="6.35" rot="R270"/>
 <element name="U$1" library="433LIB" package="BUTTON" value="BUTTON" x="6.35" y="34.29" rot="R90"/>
 <element name="U$2" library="433LIB" package="BUTTON" value="BUTTON" x="2.54" y="2.54"/>
 <element name="U$3" library="433LIB" package="USB-MB-H" value="USB_MINIUSB" x="44.45" y="43.18" rot="R180"/>
 <element name="U$4" library="433LIB" package="1X03" value="RESONATOR" x="3.81" y="15.24" rot="R270"/>
-<element name="U$5" library="433LIB" package="TO92" value="MCP1702" x="45.72" y="12.7" rot="R270"/>
+<element name="U$5" library="433LIB" package="TO92" value="MCP1702" x="41.91" y="8.89" rot="R270"/>
 <element name="U$6" library="433LIB" package="1X05" value="SLIDE_SWITCH" x="44.45" y="25.4" rot="R90"/>
 </elements>
@@
 <contactref element="U$1" pad="3"/>
 <contactref element="J1" pad="1"/>
-<wire x1="11.43" y1="39.37" x2="22.86" y2="38.1" width="0" layer="19" extent="1-1"/>
-<wire x1="11.43" y1="25.4" x2="11.43" y2="39.37" width="0" layer="19" extent="1-1"/>
-<wire x1="6.35" y1="39.37" x2="11.43" y2="39.37" width="0" layer="19" extent="1-1"/>
+<wire x1="22.86" y1="38.1" x2="21.59" y2="44.45" width="0" layer="19" extent="1-1"/>
+<wire x1="11.43" y1="44.45" x2="21.59" y2="44.45" width="0" layer="19" extent="1-1"/>
+<wire x1="6.35" y1="39.37" x2="11.43" y2="44.45" width="0" layer="19" extent="1-1"/>
 </signal>
 <signal name="+3V3">
@@
 <wire x1="20.32" y1="3.81" x2="19.05" y2="2.54" width="0.4064" layer="16"/>
 <wire x1="16.51" y1="20.32" x2="11.43" y2="20.32" width="0.4064" layer="16"/>
+<wire x1="24.13" y1="44.45" x2="33.02" y2="38.1" width="0" layer="19" extent="1-1"/>
+<wire x1="19.05" y1="44.45" x2="24.13" y2="44.45" width="0" layer="19" extent="1-1"/>
+<wire x1="16.51" y1="46.99" x2="19.05" y2="44.45" width="0" layer="19" extent="1-1"/>
 <wire x1="33.02" y1="25.4" x2="33.02" y2="38.1" width="0" layer="19" extent="1-1"/>
-<wire x1="19.05" y1="39.37" x2="33.02" y2="38.1" width="0" layer="19" extent="1-1"/>
-<wire x1="13.97" y1="43.18" x2="19.05" y2="39.37" width="0" layer="19" extent="1-1"/>
-<wire x1="11.43" y1="27.94" x2="19.05" y2="39.37" width="0" layer="19" extent="1-1"/>
-<wire x1="11.43" y1="20.32" x2="11.43" y2="27.94" width="0" layer="19" extent="1-1"/>
+<wire x1="16.51" y1="20.32" x2="33.02" y2="25.4" width="0" layer="19" extent="1-1"/>
 <wire x1="22.86" y1="7.62" x2="16.51" y2="20.32" width="0" layer="19" extent="1-1"/>
 </signal>
@@
 <contactref element="J1" pad="5"/>
 <contactref element="IC1" pad="5"/>
-<wire x1="11.43" y1="35.56" x2="22.86" y2="27.94" width="0" layer="19" extent="1-1"/>
+<wire x1="22.86" y1="27.94" x2="31.75" y2="44.45" width="0" layer="19" extent="1-1"/>
 </signal>
 <signal name="N$7">
 <contactref element="J1" pad="4"/>
 <contactref element="IC1" pad="4"/>
-<wire x1="11.43" y1="33.02" x2="22.86" y2="30.48" width="0" layer="19" extent="1-1"/>
+<wire x1="22.86" y1="30.48" x2="29.21" y2="44.45" width="0" layer="19" extent="1-1"/>
 </signal>
 <signal name="N$11">
 <contactref element="IC1" pad="20"/>
 <contactref element="C1" pad="+"/>
-<wire x1="45.72" y1="2.54" x2="31.75" y2="2.54" width="0.4064" layer="16"/>
+<wire x1="38.1" y1="2.54" x2="31.75" y2="2.54" width="0.4064" layer="16"/>
 <wire x1="31.75" y1="2.54" x2="30.48" y2="3.81" width="0.4064" layer="16"/>
 <wire x1="30.48" y1="3.81" x2="30.48" y2="16.51" width="0.4064" layer="16"/>
@@
 <contactref element="LED2" pad="K"/>
 <contactref element="R4" pad="2"/>
-<wire x1="3.81" y1="48.26" x2="13.97" y2="48.26" width="0" layer="19" extent="1-1"/>
+<wire x1="44.45" y1="2.54" x2="46.99" y2="2.54" width="0.4064" layer="16"/>
 </signal>
 <signal name="N$10">
@@
 <wire x1="46.99" y1="19.05" x2="46.99" y2="25.4" width="0.4064" layer="16"/>
 <wire x1="46.99" y1="25.4" x2="44.45" y2="27.94" width="0.4064" layer="16"/>
-<wire x1="44.45" y1="27.94" x2="47.625" y2="12.7" width="0" layer="19" extent="1-1"/>
+<wire x1="43.815" y1="8.89" x2="46.99" y2="12.065" width="0.4064" layer="16"/>
+<wire x1="46.99" y1="12.065" x2="46.99" y2="19.05" width="0.4064" layer="16"/>
 </signal>
 <signal name="N$13">
@@
 <contactref element="LED2" pad="A"/>
 <contactref element="U$5" pad="3"/>
-<wire x1="3.81" y1="45.72" x2="45.72" y2="11.43" width="0" layer="19" extent="1-1"/>
+<wire x1="41.91" y1="2.54" x2="41.91" y2="7.62" width="0.4064" layer="16"/>
 </signal>
 <signal name="N$12">
@@
 <wire x1="46.99" y1="29.21" x2="45.72" y2="29.21" width="0.4064" layer="16"/>
 <wire x1="45.72" y1="29.21" x2="44.45" y2="30.48" width="0.4064" layer="16"/>
-<wire x1="44.45" y1="33.02" x2="39.35" y2="41.58" width="0" layer="19" extent="1-1"/>
+<wire x1="39.35" y1="41.58" x2="41.91" y2="39.02" width="0.4064" layer="16"/>
+<wire x1="41.91" y1="39.02" x2="41.91" y2="35.56" width="0.4064" layer="16"/>
+<wire x1="41.91" y1="35.56" x2="44.45" y2="33.02" width="0.4064" layer="16"/>
 </signal>
 </signals>
